File: co2_7seg.kicad_sch (KiCad schematic)
At the start: 45 parts, among them J1 Conn_01x02, J2 Conn_02x03_Odd_Even, J3 Conn_01x02, Q1 2N3906, Q2 2N3906, Q3 2N3904, SW1 SW_Push, U1 ATmega328P-A, U3 MAX7221xNG, U4 MIC5205-5.0YM5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

Commit message: add reference to footprint libs, add BOM
Parts:
- C1, C2: Digikey (none) -> https://www.digikey.com/en/products/detail/kemet/C0805C180M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
- C10, C3: Digikey (none) -> https://www.digikey.com/en/products/detail/yageo/CC0805KRX7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
- C11, C12, C14: Digikey (none) -> https://www.digikey.com/en/products/detail/kyocera-avx/F921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
- C13, C15, C4, C5, C6, C7, C8, C9: Digikey (none) -> https://www.digikey.com/en/products/detail/samsung-electro-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
- J3: Digikey (none) -> https://www.digikey.com/en/products/detail/mpd-memory-prote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
- LED1, LED2, LED3, LED4: Digikey (none) -> https://www.digikey.com/en/products/detail/lumex-opto-compo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
- Q1, Q2: Digikey (none) -> https://www.digikey.com/en/products/detail/onsemi/2N3906BU/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
- Q3: Digikey (none) -> https://www.digikey.com/en/products/detail/onsemi/2N3904BU/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
- R1, R10, R11, R12, R4, R5, R6, R8: Digikey (none) -> https://www.digikey.com/en/products/detail/yageo/RC0805FR-0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
- R2, R3: Digikey (none) -> https://www.digikey.com/en/products/detail/panasonic-electr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
- R7: Digikey (none) -> https://www.digikey.com/en/products/detail/advanced-photoni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
- R9: Digikey (none) -> https://www.digikey.com/en/products/detail/stackpole-electr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
- SW1: Digikey (none) -> https://www.digikey.com/en/products/detail/c-k/RS-187R05A2-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
- U1, U4, U5: Digikey (none) -> https://www.digikey.com/en/products/detail/microchip-techno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
- U2: Digikey (none) -> https://www.digikey.com/en/products/detail/adafruit-industr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
- U3: Digikey (none) -> https://www.digikey.com/en/products/detail/analog-devices-i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
- Y1: Digikey (none) -> https://www.digikey.com/en/products/detail/ecs-inc/ECS-160-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
